Commit message: add Reaching3D task and a training example

File: python/social_bot/models/kuka_lwr_4plus/model.urdf (robot description, URDF)
Before this commit: robot kuka_lwr_4plus, 9 links, 8 joints
Links:
- removed link lwr_arm_7_link
Joints:
- removed joint lwr_arm_6_joint

Commit message: add gripper

File: python/social_bot/models/kuka_lwr_4plus/model.urdf (robot description, URDF)
Before this commit: robot kuka_lwr_4plus, 8 links, 7 joints
Links:
- added link lwr_arm_finger_l_link, mass 1.0; collision mesh filename=model://youbot/meshes/gripper/finger.stl scale=2.5 2.5 2.5; visual mesh filename=model://youbot/meshes/gripper/finger_convex.stl scale=2.5 2.5 2.5
- added link lwr_arm_finger_r_link, mass 1.0; collision mesh filename=model://youbot/meshes/gripper/finger.stl scale=2.5 2.5 2.5; visual mesh filename=model://youbot/meshes/gripper/finger_convex.stl scale=2.5 2.5 2.5
Joints:
- added joint lwr_arm_finger_l_joint: type revolute, parent lwr_arm_6_link, child lwr_arm_finger_l_link, origin xyz=0 0.1 0.1 rpy=0 0 0, axis 0 -1 0, limit lower=-2.09439510239 upper=2.09439510239 effort=200 velocity=3.14159265359
- added joint lwr_arm_finger_r_joint: type revolute, parent lwr_arm_6_link, child lwr_arm_finger_r_link, origin xyz=0 -0.1 0.1 rpy=0 0 0, axis 0 -1 0, limit lower=-2.09439510239 upper=2.09439510239 effort=200 velocity=3.14159265359
